File: hw/ECE445L_Starter/pcb_operator/ECE445L_Starter.kicad_pcb (KiCad board)
At the start: 2 copper layers, 164.2 x 114.8 mm, 66 parts, among them IC1 TLV5616, IC2 LM4041CILPR, IC3 MCP1755T-5002E_OT, J1 Speaker, J2 JTAG, J3 Battery, SW1 UP, SW2 DOWN, SW3 Reset, U103 Adafruit ST7735R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

Commit message: pedal ADC code to TM4C
Parts:
- added U7: LM2937xMP, Package_TO_SOT_SMD:SOT-223-3_TabPin2, F.Cu at (72.8, 64.2)
Connections:
- BT1 pad +: +5V -> /12V
- BT1 pad -: Net-(IC3-VIN) -> GND
- C1 pad 1: PC5 -> PB5
- C1 pad 2: +5V -> GND
- C10 pad 2: +5V -> GND
- C11 pad 2: +5V -> GND
- C12 pad 2: +5V -> GND
- C13 pad 2: +5V -> GND
- C14 pad 2: +5V -> GND
- C15 pad 2: +5V -> GND
- C16 pad 2: +5V -> GND
- C19 pad 1: Net-(IC3-VIN) -> /12V
- C19 pad 2: +5V -> GND
- C2 pad 1: PC4 -> PB3
- C2 pad 2: +5V -> GND
- C21 pad 2: +5V -> GND
- C23 pad 2: +5V -> GND
- C24 pad 1: +5V -> GND
- C25 pad 2: +5V -> GND
- C3 pad 2: +5V -> GND
- C4 pad 2: +5V -> GND
- C5 pad 2: +5V -> GND
- C6 pad 2: +5V -> GND
- C7 pad 2: +5V -> GND
- C8 pad 2: +5V -> GND
- C9 pad 2: +5V -> GND
- IC1 pad 3: +5V -> GND
- IC1 pad 5: +5V -> GND
- IC2 pad 3: +5V -> GND
- IC3 pad 1: Net-(IC3-VIN) -> /12V
- IC3 pad 2: +5V -> GND
- IC3 pad 3: +5V -> /12V
- IC3 pad 4: +5V -> unconnected-(IC3-PWRGD-Pad4)
- IC3 pad 5: unconnected-(IC3-VOUT-Pad5) -> +5V
- J2 pad 1: +5V -> GND
- R1 pad 2: PC4 -> PB3
- R2 pad 2: PC5 -> PB5
- R9 pad 2: +5V -> GND
- SW1 pad 1: +5V -> GND
- SW1 pad 2: PC4 -> PB3
- SW2 pad 1: +5V -> GND
- SW2 pad 2: PC5 -> PB5
- SW3 pad 1: +5V -> GND
- U1 pad 1: +5V -> +3V3
- U1 pad 17: +5V -> GND
- U1 pad 2: unconnected-(U1-GND-Pad2) -> GND
- U103 pad 1: +5V -> GND
- U2 pad 12: +5V -> GND
- U2 pad 27: +5V -> GND
- U2 pad 3: +5V -> GND
- U2 pad 34: +5V -> GND
- U2 pad 35: +5V -> GND
- U2 pad 39: +5V -> GND
- U2 pad 55: +5V -> GND
- U4 pad 1: +5V -> GND
- U4 pad 7: +5V -> GND
- U5 pad J1_1: Net-(U5-+3.3V) -> unconnected-(U5-+3.3V-PadJ1_1)
- U5 pad J2_1: +5V -> GND
- U5 pad J3_1: Net-(U5-+VBUS) -> +5V
- U5 pad J3_2: +5V -> GND
- VR1 pad 1: +5V -> GND
- VR2 pad 1: +5V -> GND
- VR3 pad 1: +5V -> GND
Routing:
- net GND: track 0.00 -> 588.5 mm, vias 0 -> 10
- net PB5: track 0.00 -> 192.6 mm, vias 0 -> 2
- net +5V: track 835.4 -> 939.9 mm, vias 48 -> 49
- net /12V: track 0.00 -> 89.7 mm, vias 0 -> 1
- net PB3: track 0.00 -> 82.4 mm, vias 0 -> 1
- net +3V3: track 464.3 -> 538.1 mm
- net PC5: track 267.1 -> 274.4 mm, vias 8 -> 9
- net PC4: track 259.0 -> 266.2 mm
- net /LDO: track 79.4 -> 82.0 mm
- net /+3_7V: track 138.9 -> 141.3 mm
- net PE2: track 184.2 -> 186.1 mm
