File: hw/ECE445L_Starter/pcb_operator/ECE445L_Starter.kicad_sch (KiCad schematic)
At the start: 66 parts, among them IC1 TLV5616, IC2 LM4041CILPR, IC3 MCP1755T-5002E_OT, J1 Speaker, J2 JTAG, J3 Battery, SW1 UP, SW2 DOWN, SW3 Reset, U103 Adafruit ST7735R, U2 TM4C123GH6PMIR, U3 LP2950-33LPRE3, U4 MCP34119P, U5 EK-TM4C123GXL, Y1 ABM3-16.000MHZ-B2-T

Commit message: pedal ADC code to TM4C
Parts:
- removed C17, C18, C27: 4.7uF, ECE445L:CP_Radial_Tantal200mil, symbol ECE445L:C_Polarized
- removed C20: 1u, ECE445L:C_Axial_200mil, symbol ECE445L:C
- removed J3: Battery, ECE445L:PinHeader_1x02_P2.54mm_Vertical, symbol ECE445L:Header_2
- removed TP3: 3.7V, ECE445L:Testpoint_1x02_P2.54mm, symbol Connector:TestPoint
- removed TP5: +3.7V, ECE445L:Testpoint_1x02_P2.54mm, symbol ECE445L:Testpoint
- removed TP6: GND, ECE445L:Testpoint_1x02_P2.54mm, symbol ECE445L:Testpoint
- removed TP7: +3.3V, ECE445L:Testpoint_1x02_P2.54mm, symbol ECE445L:Testpoint
- removed TP8: 3.3V, ECE445L:Testpoint_1x02_P2.54mm, symbol Connector:TestPoint
- removed U3: LP2950-33LPRE3, ECE445L:TL431CLPM, symbol ECE445L:LP2950-33LPRE3
- added C29: 10uF, ECE445L:C_Axial_200mil, symbol ECE445L:C
- added C30: 22uF, ECE445L:C_Axial_200mil, symbol ECE445L:C
- added TP11: +3.3V, ECE445L:Testpoint_1x02_P2.54mm, symbol ECE445L:Testpoint
- added TP12: 3.3V, ECE445L:Testpoint_1x02_P2.54mm, symbol Connector:TestPoint
- added U7: LM2937xMP, Package_TO_SOT_SMD:SOT-223-3_TabPin2, symbol Regulator_Linear:LM2937xMP
Connections:
- net +3V3: now also U1.1 (VIN), C30.1, TP11.1 (A), TP11.2 (B), TP12.1, U7.3 (VO)
- net +5V: now also IC3.5 (VOUT), U5.J3_1 (+VBUS), C29.1, U7.1 (VI); no longer BT1.+, C1.2, C10.2, C11.2, C12.2, C13.2, C14.2, C15.2, C16.2, C19.2, C2.2, C21.2, C23.2, C24.1, C25.2, C26.2, C3.2, C4.2, C5.2, C6.2, C7.2, C8.2, C9.2, IC1.3 (~{CS}), IC1.5 (AGND), IC2.3, IC3.2 (GND), IC3.3 (~{SHDN}), IC3.4 (PWRGD), J2.1 (A), R9.2, SW1.1, SW2.1, SW3.1, U1.1 (VIN), U1.17 (GND), U103.1 (GND), U2.12 (GND_1), U2.27 (GND_2), U2.3 (GNDA), U2.34 (XOSC0), U2.35 (GNDX), U2.39 (GND_3), U2.55 (GND_4), U4.1 (CD), U4.7 (GND), U5.J2_1 (GND), U5.J3_2 (GND), VR1.1, VR2.1, VR3.1
- net PB3: now also C2.1, R1.2, SW1.2
- net PB5: now also C1.1, R2.2, SW2.2
- net PC4: no longer C2.1, R1.2, SW1.2
- net PC5: no longer C1.1, R2.2, SW2.2
- net 12V: now reaches C19.1, IC3.1 (VIN)
- net 12V: now also BT1.+, IC3.3 (~{SHDN}); no longer BT1.-
- net GND: now reaches U1.2 (GND)
- net GND: now also BT1.-, C1.2, C10.2, C11.2, C12.2, C13.2, C14.2, C15.2, C16.2, C19.2, C2.2, C21.2, C23.2, C24.1, C25.2, C26.2, C3.2, C4.2, C5.2, C6.2, C7.2, C8.2, C9.2, IC1.3 (~{CS}), IC1.5 (AGND), IC2.3, IC3.2 (GND), J2.1 (A), R9.2, SW1.1, SW2.1, SW3.1, U1.17 (GND), U103.1 (GND), U2.12 (GND_1), U2.27 (GND_2), U2.3 (GNDA), U2.34 (XOSC0), U2.35 (GNDX), U2.39 (GND_3), U2.55 (GND_4), U4.1 (CD), U4.7 (GND), U5.J2_1 (GND), U5.J3_2 (GND), VR1.1, VR2.1, VR3.1, C29.2, C30.2, U7.2 (GND)
- no-connect marks 6 -> 7
Other:
- moved on the sheet: BT1, C1, C10, C11, C12, C13, C14, C15, C16, C19, C2, C3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
